Commit message: ssmm_gazebo urdf and launch

File: ssmm_gazebo/urdf/3dof.urdf (robot description, URDF)
Before this commit: robot ssmm, 1 links, 0 joints
Links:
- link base_link: mass None -> 0.8861; geometry collision mesh filename=package://ssmm_gazebo/meshes/base_link.STL; visual mesh filename=package://ssmm_gazebo/meshes/base_link.STL
