Commit message: little change

File: ssmm_gazebo/urdf/ssmm.urdf (robot description, URDF)
Before this commit: robot ssmm, 1 links, 0 joints
Links:
- link base_link: geometry collision cylinder length=0.6 radius=0.2; visual cylinder length=0.6 radius=0.2

Commit message: mobile urdf changed

File: ssmm_gazebo/urdf/ssmm.urdf (robot description, URDF)
Before this commit: robot ssmm, 1 links, 0 joints
Links:
- added link left_wheel, mass 0.1112; collision mesh filename=package://ssmm_gazebo/meshes/left_wheel.STL; visual mesh filename=package://ssmm_gazebo/meshes/left_wheel.STL
- added link right_wheel, mass 0.111202201176881; collision mesh filename=package://ssmm_gazebo/meshes/right_wheel.STL; visual mesh filename=package://ssmm_gazebo/meshes/right_wheel.STL
- link base_link: geometry collision mesh filename=package://ssmm_gazebo/meshes/base_link.STL; visual mesh filename=package://ssmm_gazebo/meshes/base_link.STL
Joints:
- added joint left_wheel_joint: type continuous, parent base_link, child left_wheel, origin xyz=0 0 -0.1935 rpy=0 0 2.5629, axis 0 0 0
- added joint right_wheel_joint: type continuous, parent base_link, child right_wheel, origin xyz=0 0 0.1935 rpy=3.1416 0 2.5629, axis 0 0 0, limit lower=0 upper=0 effort=0 velocity=0
