Commit message: fixing urdf mesh loading problem

File: ssmm_gazebo/urdf/ssmm_gazebo.urdf (robot description, URDF)
Before this commit: robot ssmm_gazebo, 4 links, 3 joints
Links:
- removed link left_wheel
- removed link lidar
- removed link right_wheel
- link base_link: geometry collision mesh filename=file://$(find ssmm_gazebo)/meshes/base_link.STL scale=1 1 1; visual mesh filename=file://$(find ssmm_gazebo)/meshes/base_link.STL scale=1 1 1
Joints:
- removed joint base_to_lidar
- removed joint base_to_lw
- removed joint base_to_rw

Commit message: xacro, urdf added

File: ssmm_gazebo/urdf/ssmm_gazebo.urdf (robot description, URDF)
Before this commit: robot ssmm_gazebo, 4 links, 3 joints
Links:
- link base_link: geometry collision mesh filename=file:///home/benlee/ros2_ws/install/ssmm_gazebo/share/ssmm_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 scale=1 1 1; visual mesh filename=file:///home/benlee/ros2_ws/install/ssmm_gazebo/share/ssmm_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 scale=1 1 1
- link left_wheel: geometry collision mesh filename=file:///home/benlee/ros2_ws/install/ssmm_gazebo/share/ssmm_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; visual mesh filename=file:///home/benlee/ros2_ws/install/ssmm_gazebo/share/ssmm_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
- link lidar: geometry collision mesh filename=file:///home/benlee/ros2_ws/install/ssmm_gazebo/share/ssmm_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; visual mesh filename=file:///home/benlee/ros2_ws/install/ssmm_gazebo/share/ssmm_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
- link right_wheel: geometry collision mesh filename=file:///home/benlee/ros2_ws/install/ssmm_gazebo/share/ssmm_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; visual mesh filename=file:///home/benlee/ros2_ws/install/ssmm_gazebo/share/ssmm_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

Commit message: new model urdf update

File: ssmm_gazebo/urdf/ssmm_gazebo.urdf (robot description, URDF)
Before this commit: robot ssmm_gazebo, 4 links, 3 joints
Joints:
- joint base_to_lw: origin xyz=0.10789 0.175 0.025 rpy=1.5708 0 3.1416 -> xyz=0.106 0.17775 0.022 rpy=1.5708 0 3.1416
- joint base_to_rw: origin xyz=0.10789 -0.175 0.025 rpy=1.5708 0 0 -> xyz=0.106 -0.17775 0.022 rpy=1.5708 0 0
