Commit message: new ssmm_robot urdf added

File: ssmm_gazebo/urdf/ssmm_gazebo.urdf.xacro (robot description, xacro)
@@ -3,6 +3,6 @@
      Commit Version: 1.5.1-0-g916b5db  Build Version: 1.5.7152.31018
      For more information, please see http://wiki.ros.org/sw_urdf_exporter -->
-<robot name="ssmm_gazebo" xmlns:xacro="http://www.ros.org/wiki/xacro">
-  <xacro:include filename="$(find ssmm_gazebo)/urdf/ssmm_gazebo.gazebo"/>
+<robot name="ssmm_robot" xmlns:xacro="http://www.ros.org/wiki/xacro">
+  <xacro:include filename="$(find ssmm_robot)/urdf/ssmm_robot.gazebo"/>
   <link name="base_link">
     <inertial>
@@ -25,5 +25,5 @@
         rpy="1.5708 0 0" />
       <geometry>
-        <mesh filename="file://$(find ssmm_gazebo)/meshes/base_link.STL" scale = "1 1 1"/>
+        <mesh filename="file://$(find ssmm_robot)/meshes/base_link.STL" scale = "1 1 1"/>
       </geometry>
       <material
@@ -39,5 +39,5 @@
       <geometry>
         <mesh
-          filename="file://$(find ssmm_gazebo)/meshes/base_link.STL" scale = "1 1 1"/>
+          filename="file://$(find ssmm_robot)/meshes/base_link.STL" scale = "1 1 1"/>
       </geometry>
     </collision>
@@ -64,5 +64,5 @@
       <geometry>
         <mesh
-          filename="file://$(find ssmm_gazebo)/meshes/right_wheel.STL" />
+          filename="file://$(find ssmm_robot)/meshes/right_wheel.STL" />
       </geometry>
       <material
@@ -78,5 +78,5 @@
       <geometry>
         <mesh
-          filename="file://$(find ssmm_gazebo)/meshes/right_wheel.STL" />
+          filename="file://$(find ssmm_robot)/meshes/right_wheel.STL" />
       </geometry>
     </collision>
@@ -114,5 +114,5 @@
       <geometry>
         <mesh
-          filename="file://$(find ssmm_gazebo)/meshes/left_wheel.STL" />
+          filename="file://$(find ssmm_robot)/meshes/left_wheel.STL" />
       </geometry>
       <material
@@ -128,5 +128,5 @@
       <geometry>
         <mesh
-          filename="file://$(find ssmm_gazebo)/meshes/left_wheel.STL" />
+          filename="file://$(find ssmm_robot)/meshes/left_wheel.STL" />
       </geometry>
     </collision>
@@ -165,5 +165,5 @@
       <geometry>
         <mesh
-          filename="file://$(find ssmm_gazebo)/meshes/lidar.STL" />
+          filename="file://$(find ssmm_robot)/meshes/lidar.STL" />
       </geometry>
       <material
@@ -179,5 +179,5 @@
       <geometry>
         <mesh
-          filename="file://$(find ssmm_gazebo)/meshes/lidar.STL" />
+          filename="file://$(find ssmm_robot)/meshes/lidar.STL" />
       </geometry>
     </collision>

File: ssmm_robot/urdf/ssmm_robot.urdf (robot description, URDF)
Before this commit: robot ssmm_robot, 13 links, 12 joints
Links:
- link base_link: geometry collision mesh filename=file:///home/benlee/ros2_ws/install/ssmm_robot/share/ssmm_r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; visual mesh filename=file:///home/benlee/ros2_ws/install/ssmm_robot/share/ssmm_r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
- link cam: geometry collision mesh filename=file:///home/benlee/ros2_ws/install/ssmm_robot/share/ssmm_r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; visual mesh filename=file:///home/benlee/ros2_ws/install/ssmm_robot/share/ssmm_r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
- link cam_bracket: geometry collision mesh filename=file:///home/benlee/ros2_ws/install/ssmm_robot/share/ssmm_r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; visual mesh filename=file:///home/benlee/ros2_ws/install/ssmm_robot/share/ssmm_r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
- link cam_link1: geometry collision mesh filename=file:///home/benlee/ros2_ws/install/ssmm_robot/share/ssmm_r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; visual mesh filename=file:///home/benlee/ros2_ws/install/ssmm_robot/share/ssmm_r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
- link cam_link2: geometry collision mesh filename=file:///home/benlee/ros2_ws/install/ssmm_robot/share/ssmm_r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; visual mesh filename=file:///home/benlee/ros2_ws/install/ssmm_robot/share/ssmm_r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
- link caster: geometry collision mesh filename=file:///home/benlee/ros2_ws/install/ssmm_robot/share/ssmm_r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; visual mesh filename=file:///home/benlee/ros2_ws/install/ssmm_robot/share/ssmm_r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
- link left_finger: geometry collision mesh filename=file:///home/benlee/ros2_ws/install/ssmm_robot/share/ssmm_r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; visual mesh filename=file:///home/benlee/ros2_ws/install/ssmm_robot/share/ssmm_r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
- link left_wheel: geometry collision mesh filename=file:///home/benlee/ros2_ws/install/ssmm_robot/share/ssmm_r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; visual mesh filename=file:///home/benlee/ros2_ws/install/ssmm_robot/share/ssmm_r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
- link lidar: geometry collision mesh filename=file:///home/benlee/ros2_ws/install/ssmm_robot/share/ssmm_r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; visual mesh filename=file:///home/benlee/ros2_ws/install/ssmm_robot/share/ssmm_r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
- link link1: geometry collision mesh filename=file:///home/benlee/ros2_ws/install/ssmm_robot/share/ssmm_r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; visual mesh filename=file:///home/benlee/ros2_ws/install/ssmm_robot/share/ssmm_r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
- link link2: geometry collision mesh filename=file:///home/benlee/ros2_ws/install/ssmm_robot/share/ssmm_r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; visual mesh filename=file:///home/benlee/ros2_ws/install/ssmm_robot/share/ssmm_r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
- link link3: geometry collision mesh filename=file:///home/benlee/ros2_ws/install/ssmm_robot/share/ssmm_r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; visual mesh filename=file:///home/benlee/ros2_ws/install/ssmm_robot/share/ssmm_r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
- link right_wheel: geometry collision mesh filename=file:///home/benlee/ros2_ws/install/ssmm_robot/share/ssmm_r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; visual mesh filename=file:///home/benlee/ros2_ws/install/ssmm_robot/share/ssmm_r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
