Commit message: description and bringup pkg added

File: ssmm_description/urdf/ssmm_gazebo.urdf.xacro (robot description, xacro)
@@ -3,21 +3,58 @@
      Commit Version: 1.5.1-0-g916b5db  Build Version: 1.5.7152.31018
      For more information, please see http://wiki.ros.org/sw_urdf_exporter -->
-<robot
-  name="ssmm_gazebo">
-  <link
-    name="base_link">
+<robot name="ssmm_gazebo" xmlns:xacro="http://www.ros.org/wiki/xacro">
+  <xacro:include filename="$(find ssmm_gazebo)/urdf/ssmm_gazebo.gazebo"/>
+  <link name="base_link">
     <inertial>
       <origin
-        xyz="0.043579 -0.017838 -0.022157"
+        xyz="0.0054761 0.046718 -0.00077332"
         rpy="0 0 0" />
       <mass
-        value="0.8861" />
+        value="2.2263" />
       <inertia
-        ixx="0.0079901"
-        ixy="1.1902E-06"
-        ixz="-1.0289E-18"
-        iyy="0.016382"
-        iyz="-4.3652E-19"
-        izz="0.0084009" />
+        ixx="0.021054"
+        ixy="1.5769E-06"
+        ixz="-0.00021664"
+        iyy="0.036188"
+        iyz="-7.2302E-08"
+        izz="0.016028" />
+    </inertial>
+    <visual>
+      <origin
+        xyz="0 0 0"
+        rpy="1.5708 0 0" />
+      <geometry>
+        <mesh filename="file://$(find ssmm_gazebo)/meshes/base_link.STL" scale = "1 1 1"/>
+      </geometry>
+      <material
+        name="">
+        <color
+          rgba="0.75294 0.75294 0.75294 1" />
+      </material>
+    </visual>
+    <collision>
+      <origin
+        xyz="0 0 0"
+        rpy="1.5708  0 0" />
+      <geometry>
+        <mesh
+          filename="file://$(find ssmm_gazebo)/meshes/base_link.STL" scale = "1 1 1"/>
+      </geometry>
+    </collision>
+  </link>
+  <link name="right_wheel">
+    <inertial>
+      <origin
+        xyz="0 1.7347E-18 0"
+        rpy="0 0 0" />
+      <mass
+        value="0.1112" />
+      <inertia
+        ixx="5.5328E-05"
+        ixy="-1.0735E-21"
+        ixz="-3.2923E-19"
+        iyy="5.5328E-05"
+        iyz="-2.9102E-21"
+        izz="0.00010246" />
     </inertial>
     <visual>
@@ -27,5 +64,5 @@
       <geometry>
         <mesh
-          filename="package://ssmm_gazebo/meshes/base_link.STL" />
+          filename="file://$(find ssmm_gazebo)/meshes/right_wheel.STL" />
       </geometry>
       <material
@@ -41,23 +78,33 @@
       <geometry>
         <mesh
-          filename="package://ssmm_gazebo/meshes/base_link.STL" />
+          filename="file://$(find ssmm_gazebo)/meshes/right_wheel.STL" />
       </geometry>
     </collision>
   </link>
-  <link
-    name="right_wheel">
+  <joint name="base_to_rw" type="continuous">
+    <origin
+      xyz="0.10789 -0.175 0.025"
+      rpy="1.5708 0 0" />
+    <parent
+      link="base_link" />
+    <child
+      link="right_wheel" />
+    <axis
+      xyz="0 0 1" />
+  </joint>
+  <link name="left_wheel">
     <inertial>
       <origin
-        xyz="0.12573 0.19245 0.13898"
+        xyz="-2.9803E-14 -2.681E-14 1.5599E-14"
         rpy="0 0 0" />
       <mass
-        value="0.11659" />
+        value="0.1112" />
       <inertia
-        ixx="5.5634E-05"
-        ixy="-6.5495E-10"
-        ixz="-1.1058E-09"
-        iyy="5.5634E-05"
-        iyz="6.7403E-10"
-        izz="0.00010273" />
+        ixx="5.5328E-05"
+        ixy="-1.3032E-22"
+        ixz="-4.1548E-19"
+        iyy="5.5328E-05"
+        iyz="-1.6842E-19"
+        izz="0.00010246" />
     </inertial>
     <visual>
@@ -67,5 +114,5 @@
       <geometry>
         <mesh
-          filename="package://ssmm_gazebo/meshes/right_wheel.STL" />
+          filename="file://$(find ssmm_gazebo)/meshes/left_wheel.STL" />
       </geometry>
       <material
@@ -81,67 +128,12 @@
       <geometry>
         <mesh
-          filename="package://ssmm_gazebo/meshes/right_wheel.STL" />
+          filename="file://$(find ssmm_gazebo)/meshes/left_wheel.STL" />
       </geometry>
     </collision>
   </link>
-  <joint
-    name="base_to_rw"
-    type="continuous">
+  <joint name="base_to_lw" type="continuous">
     <origin
-      xyz="0.10602 -0.183 0.022"
-      rpy="1.5708 0 0" />
-    <parent
-      link="base_link" />
-    <child
-      link="right_wheel" />
-    <axis
-      xyz="0 0 1" />
-  </joint>
-  <link
-    name="left_wheel">
-    <inertial>
-      <origin
-        xyz="-0.12573 0.19245 0.13898"
-        rpy="0 0 0" />
-      <mass
-        value="0.11659" />
-      <inertia
-        ixx="5.5634E-05"
-        ixy="6.9199E-10"
-        ixz="-1.0614E-09"
-        iyy="5.5634E-05"
-        iyz="-7.4188E-10"
-        izz="0.00010273" />
-    </inertial>
-    <visual>
-      <origin
-        xyz="0 0 0"
-        rpy="0 0 0" />
-      <geometry>
-        <mesh
-          filename="package://ssmm_gazebo/meshes/left_wheel.STL" />
-      </geometry>
-      <material
-        name="">
-        <color
-          rgba="0.75294 0.75294 0.75294 1" />
-      </material>
-    </visual>
-    <collision>
-      <origin
-        xyz="0 0 0"
-        rpy="0 0 0" />
-      <geometry>
-        <mesh
-          filename="package://ssmm_gazebo/meshes/left_wheel.STL" />
-      </geometry>
-    </collision>
-  </link>
-  <joint
-    name="base_to_lw"
-    type="continuous">
-    <origin
-      xyz="0.10602 0.183 0.022"
-      rpy="-1.5708 0 0" />
+      xyz="0.10789 0.175 0.025"
+      rpy="1.5708 0 3.1416" />
     <parent
       link="base_link" />
@@ -155,15 +147,15 @@
     <inertial>
       <origin
-        xyz="-0.13583 -0.060836 -0.10229"
+        xyz="0 0 0"
         rpy="0 0 0" />
       <mass
-        value="0.16306" />
+        value="0" />
       <inertia
-        ixx="6.0724E-05"
-        ixy="4.1104E-08"
-        ixz="2.464E-07"
-        iyy="9.2342E-05"
-        iyz="6.7628E-08"
-        izz="7.5686E-05" />
+        ixx="0"
+        ixy="0"
+        ixz="0"
+        iyy="0"
+        iyz="0"
+        izz="0" />
     </inertial>
     <visual>
@@ -173,10 +165,10 @@
       <geometry>
         <mesh
-          filename="package://ssmm_gazebo/meshes/lidar.STL" />
+          filename="file://$(find ssmm_gazebo)/meshes/lidar.STL" />
       </geometry>
       <material
         name="">
         <color
-          rgba="0.75294 0.75294 0.75294 1" />
+          rgba="1 1 1 1" />
       </material>
     </visual>
@@ -187,14 +179,12 @@
       <geometry>
         <mesh
-          filename="package://ssmm_gazebo/meshes/lidar.STL" />
+          filename="file://$(find ssmm_gazebo)/meshes/lidar.STL" />
       </geometry>
     </collision>
   </link>
-  <joint
-    name="base_to_lidar"
-    type="fixed">
+  <joint name="base_to_lidar" type="fixed">
     <origin
-      xyz="0.10202 0 0.1339"
-      rpy="0 0 0" />
+      xyz="0.097808 -0.0015 0.13"
+      rpy="1.5708 0 0" />
     <parent
       link="base_link" />
