Commit message: Solving NaN input to TF by setting Axis in urdf

File: ssmm_robot/urdf/ssmm_robot.urdf (robot description, URDF)
Before this commit: robot ssmm_robot, 13 links, 12 joints
Joints:
- joint base_to_link1: axis 0 0 0 -> 0 0 1
- joint cam_link1_to_link2: axis 0 0 0 -> 0 0 1
- joint link1_to_link2: axis 0 0 0 -> 0 0 1
- joint link2_to_cam_bracket: axis 0 0 0 -> 0 0 1
- joint link2_to_link3: axis 0 0 0 -> 0 0 1
- joint link3_to_lf: axis 0 0 0 -> 0 0 1

Commit message: change few mesh files for urdf setting

File: ssmm_robot/urdf/ssmm_robot.urdf (robot description, URDF)
Before this commit: robot ssmm_robot, 13 links, 12 joints
Joints:
- joint base_to_cam_motor1: origin xyz=0.0013904 -0.0225 1.3186 rpy=3.1416 0 0 -> xyz=0.0023904 -0.0025 1.3186 rpy=1.5708 0 -1.5708
- joint cam_link1_to_link2: origin xyz=0 0 0 rpy=0 0 0 -> xyz=0.035 0 0.05 rpy=3.1416 1.5708 0
- joint link1_to_link2: origin xyz=0.16921 0.0066 0.06353 rpy=0 0 0 -> xyz=0.16921 0.0066 0.06353 rpy=1.5708 0 0
- joint link2_to_cam_bracket: origin xyz=0 0.019 0.0421 rpy=1.5708 0 -3.1416 -> xyz=0 0.019 0.0421 rpy=3.1416 0 -3.1416

Commit message: change corrdinate

File: ssmm_robot/urdf/ssmm_robot.urdf (robot description, URDF)
Before this commit: robot ssmm_robot, 13 links, 12 joints
Joints:
- joint link1_to_link2: origin xyz=0.16921 0.0066 0.06353 rpy=1.5708 0 0 -> xyz=0.16921 0.073 -0.013 rpy=1.5708 0 0
- joint link2_to_link3: origin xyz=0.4216 0.0079 -0.0018 rpy=1.5708 0 1.5598 -> xyz=0.4 0.005 -0.085 rpy=1.5708 0 1.5598

Commit message: left finger stl change and urdf change

File: ssmm_robot/urdf/ssmm_robot.urdf (robot description, URDF)
Before this commit: robot ssmm_robot, 13 links, 12 joints
Joints:
- joint base_to_caster: origin xyz=-0.10811 0 -0.026223 rpy=0 0 0 -> xyz=-0.10811 0.0012 -0.026223 rpy=0 0 0
- joint base_to_lidar: origin xyz=0.10389 0 0.1153 rpy=0 0 0 -> xyz=0.10389 0.0015 0.1153 rpy=0 0 0
- joint base_to_link1: origin xyz=-0.13891 -0.0395 0.20287 rpy=0 0 0 -> xyz=-0.13847 -0.04103 0.20287 rpy=0 0 0
- joint base_to_lw: origin xyz=0.10789 0.184 0.014 rpy=1.5708 0 3.1416 -> xyz=0.10991 0.1828 0.014 rpy=1.5708 0 3.1416
- joint base_to_rw: origin xyz=0.10789 -0.184 0.014 rpy=-1.5708 0 -3.1416 -> xyz=0.10991 -0.1828 0.014 rpy=-1.5708 0 -3.1416
- joint link1_to_link2: origin xyz=0.16921 0.073 -0.013 rpy=1.5708 0 0 -> xyz=0.16931 0.0 0.063 rpy=1.5708 0 0
- joint link2_to_link3: origin xyz=0.4 0.005 -0.085 rpy=1.5708 0 1.5598 -> xyz=0.42167 -0.011 -0.03 rpy=1.5708 0 1.5598
- joint link3_to_lf: origin xyz=0.0005073 0 0.045997 rpy=0 0 0 -> xyz=-0.005 -0.03 0.10983 rpy=0 0 0

Commit message: fixing URDF visual coordinate

File: ssmm_robot/urdf/ssmm_robot.urdf (robot description, URDF)
Before this commit: robot ssmm_robot, 13 links, 12 joints
Joints:
- joint base_to_cam_motor1: origin xyz=0.0023904 -0.0025 1.3186 rpy=1.5708 0 -1.5708 -> xyz=0.020904 -0.0059 1.3186 rpy=1.5708 0 -1.5708
- joint cam_link1_to_link2: origin xyz=0.035 0 0.05 rpy=3.1416 1.5708 0 -> xyz=0.055 0.0045 0.039 rpy=3.1416 1.5708 0

Commit message: URDF done

File: ssmm_robot/urdf/ssmm_robot.urdf (robot description, URDF)
Before this commit: robot ssmm_robot, 13 links, 12 joints
Joints:
- joint link2_to_cam_bracket: origin xyz=0 0.019 0.0421 rpy=3.1416 0 -3.1416 -> xyz=0.02 0.04 -0.001 rpy=3.1416 0 -3.1416
