Commit message: URDF from Fusion360

File: ssmm_robot/urdf/ssmm_robot.urdf.xacro (robot description, xacro)
@@ -257,5 +257,5 @@
       xyz="0 0 0" />
   </joint>
-  <link
+  <!-- <link
     name="link1">
     <inertial>
@@ -710,4 +710,4 @@
     <axis
       xyz="0 0 0" />
-  </joint>
+  </joint> -->
 </robot>

File: ssmm_robot/urdf/ssmm_test.urdf (robot description, URDF)
Before this commit: robot ssmm_robot, 5 links, 4 joints
Links:
- added link cam, mass 0.00015644; collision mesh filename=file:///home/benlee/ros2_ws/install/ssmm_robot/share/ssmm_r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; visual mesh filename=file:///home/benlee/ros2_ws/install/ssmm_robot/share/ssmm_r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
- added link cam_bracket, mass 0.00022031; collision mesh filename=file:///home/benlee/ros2_ws/install/ssmm_robot/share/ssmm_r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; visual mesh filename=file:///home/benlee/ros2_ws/install/ssmm_robot/share/ssmm_r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
- added link cam_link1, mass 0.00061567; collision mesh filename=file:///home/benlee/ros2_ws/install/ssmm_robot/share/ssmm_r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; visual mesh filename=file:///home/benlee/ros2_ws/install/ssmm_robot/share/ssmm_r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
- added link cam_link2, mass 0.00054378; collision mesh filename=file:///home/benlee/ros2_ws/install/ssmm_robot/share/ssmm_r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; visual mesh filename=file:///home/benlee/ros2_ws/install/ssmm_robot/share/ssmm_r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
- added link left_finger, mass 0.00015302; collision mesh filename=file:///home/benlee/ros2_ws/install/ssmm_robot/share/ssmm_r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; visual mesh filename=file:///home/benlee/ros2_ws/install/ssmm_robot/share/ssmm_r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
- added link link1, mass 0.0054731; collision mesh filename=file:///home/benlee/ros2_ws/install/ssmm_robot/share/ssmm_r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; visual mesh filename=file:///home/benlee/ros2_ws/install/ssmm_robot/share/ssmm_r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
- added link link2, mass 0.0019489; collision mesh filename=file:///home/benlee/ros2_ws/install/ssmm_robot/share/ssmm_r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; visual mesh filename=file:///home/benlee/ros2_ws/install/ssmm_robot/share/ssmm_r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
- added link link3, mass 0.0019674; collision mesh filename=file:///home/benlee/ros2_ws/install/ssmm_robot/share/ssmm_r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; visual mesh filename=file:///home/benlee/ros2_ws/install/ssmm_robot/share/ssmm_r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
Joints:
- added joint base_to_cam_motor1: type fixed, parent base_link, child cam_link1, origin xyz=0.020904 -0.0059 1.3186 rpy=1.5708 0 -1.5708, axis 0 0 0
- added joint base_to_link1: type prismatic, parent base_link, child link1, origin xyz=-0.13847 -0.04103 0.20287 rpy=0 0 0, axis 0 0 1, limit lower=0 upper=0 effort=0 velocity=0
- added joint bracket_to_cam: type fixed, parent cam_bracket, child cam, origin xyz=0 0.0559 -0.019 rpy=-1.5708 -1.5598 0, axis 0 0 0
- added joint cam_link1_to_link2: type revolute, parent cam_link1, child cam_link2, origin xyz=0.055 0.0045 0.039 rpy=3.1416 1.5708 0, axis 0 0 1, limit lower=0 upper=0 effort=0 velocity=0
- added joint link1_to_link2: type prismatic, parent link1, child link2, origin xyz=0.16931 0.0 0.063 rpy=1.5708 0 0, axis 0 0 1, limit lower=0 upper=0 effort=0 velocity=0
- added joint link2_to_cam_bracket: type revolute, parent cam_link2, child cam_bracket, origin xyz=0.02 0.04 -0.001 rpy=3.1416 0 -3.1416, axis 0 0 1, limit lower=0 upper=0 effort=0 velocity=0
- added joint link2_to_link3: type revolute, parent link2, child link3, origin xyz=0.42167 -0.011 -0.03 rpy=1.5708 0 1.5598, axis 0 0 1, limit lower=0 upper=0 effort=0 velocity=0
- added joint link3_to_lf: type prismatic, parent link3, child left_finger, origin xyz=-0.005 -0.03 0.10983 rpy=0 0 0, axis 0 0 1, limit lower=0 upper=0 effort=0 velocity=0
- joint base_to_lw: origin xyz=0.10991 0.1828 0.014 rpy=-1.5708 0 -3.1416 -> xyz=0.10991 0.1828 0.014 rpy=1.5708 0 3.1416
