Commit message: adding joint state publisher and hardware pugin

File: ssmm_robot_description/ros2_control/ssmm_robot.ros2_control.xacro (robot description, xacro)
@@ -4,14 +4,14 @@
     <ros2_control name="${name}" type="system">
       <hardware>
-        <plugin>ros2_control_demo_hardware/DiffBotSystemHardware</plugin>
+        <plugin>ssmm_robot_hardware/DiffBotSystemHardware</plugin>
         <param name="example_param_hw_start_duration_sec">0</param>
         <param name="example_param_hw_stop_duration_sec">3.0</param>
       </hardware>
-      <joint name="${prefix}left_wheel">
+      <joint name="${prefix}base_to_lw">
         <command_interface name="velocity"/>
         <state_interface name="position"/>
         <state_interface name="velocity"/>
       </joint>
-      <joint name="${prefix}right_wheel">
+      <joint name="${prefix}base_to_rw">
         <command_interface name="velocity"/>
         <state_interface name="position"/>

Commit message: manipulator_controller adding #1

File: ssmm_robot_description/ros2_control/ssmm_robot.ros2_control.xacro (robot description, xacro)
@@ -19,4 +19,39 @@
       </joint>
     </ros2_control>
+    <ros2_control name="${name}" type="system">
+      <hardware>
+        <plugin>ssmm_robot_hardware/RRBotSystemPositionOnlyHardware</plugin>
+        <param name="example_param_hw_start_duration_sec">0</param>
+        <param name="example_param_hw_stop_duration_sec">3.0</param>
+      </hardware>
+      <joint name="${prefix}link1_to_link2">
+        <command_interface name="position">
+          <param name="min">-1</param>
+          <param name="max">1</param>
+        </command_interface>
+        <state_interface name="position"/>
+      </joint>
+      <joint name="${prefix}link2_to_link3">
+        <command_interface name="position">
+          <param name="min">-1</param>
+          <param name="max">1</param>
+        </command_interface>
+        <state_interface name="position"/>
+      </joint>
+      <joint name="${prefix}link3_to_ee">
+        <command_interface name="position">
+          <param name="min">-1</param>
+          <param name="max">1</param>
+        </command_interface>
+        <state_interface name="position"/>
+      </joint>
+      <joint name="${prefix}ee_to_finger">
+        <command_interface name="position">
+          <param name="min">-1</param>
+          <param name="max">1</param>
+        </command_interface>
+        <state_interface name="position"/>
+      </joint>
+    </ros2_control>
   </xacro:macro>
 </robot>

Commit message: forwared controller added and activate success

File: ssmm_robot_description/ros2_control/ssmm_robot.ros2_control.xacro (robot description, xacro)
@@ -9,12 +9,12 @@
       </hardware>
       <joint name="${prefix}base_to_lw">
-        <command_interface name="velocity"/>
+        <command_interface name="position"/>
         <state_interface name="position"/>
-        <state_interface name="velocity"/>
+        <state_interface name="position"/>
       </joint>
       <joint name="${prefix}base_to_rw">
-        <command_interface name="velocity"/>
+        <command_interface name="position"/>
         <state_interface name="position"/>
-        <state_interface name="velocity"/>
+        <state_interface name="position"/>
       </joint>
       <joint name="${prefix}link1_to_link2">
@@ -24,7 +24,7 @@
         </command_interface>
         <state_interface name="velocity"/> -->
-        <command_interface name="velocity"/>
+        <command_interface name="position"/>
         <state_interface name="position"/>
-        <state_interface name="velocity"/>
+        <state_interface name="position"/>
       </joint>
       <joint name="${prefix}link2_to_link3">
@@ -34,7 +34,7 @@
         </command_interface>
         <state_interface name="velocity"/> -->
-        <command_interface name="velocity"/>
+        <command_interface name="position"/>
         <state_interface name="position"/>
-        <state_interface name="velocity"/>
+        <state_interface name="position"/>
       </joint>
       <joint name="${prefix}link3_to_ee">
@@ -44,7 +44,7 @@
         </command_interface>
         <state_interface name="velocity"/> -->
-        <command_interface name="velocity"/>
+        <command_interface name="position"/>
         <state_interface name="position"/>
-        <state_interface name="velocity"/>
+        <state_interface name="position"/>
       </joint>
       <joint name="${prefix}ee_to_finger">
@@ -54,7 +54,22 @@
         </command_interface>
         <state_interface name="velocity"/> -->
-        <command_interface name="velocity"/>
+        <command_interface name="position"/>
         <state_interface name="position"/>
-        <state_interface name="velocity"/>
+        <state_interface name="position"/>
+      </joint>
+      <joint name="${prefix}link1_to_cm1">
+        <command_interface name="position"/>
+        <state_interface name="position"/>
+        <state_interface name="position"/>
+      </joint>
+      <joint name="${prefix}cm1_to_cm2">
+        <command_interface name="position"/>
+        <state_interface name="position"/>
+        <state_interface name="position"/>
+      </joint>
+      <joint name="${prefix}cm2_to_cam">
+        <command_interface name="position"/>
+        <state_interface name="position"/>
+        <state_interface name="position"/>
       </joint>
     </ros2_control>
